File: PCB/choc_in_60.sch (KiCad schematic (older format))
At the start: 212 parts, among them J1 USB_C_Receptacle_USB2.0, J2 Conn_01x03, J3 Conn_01x02, J5 Conn_02x03_Odd_Even, U1 ATmega32U4-MU, U2 24LC64, U3 ATmega32U4-AU, Y1 16MHz

Commit message: 配線途中
Parts:
- removed H5: MountingHole, MountingHole:MountingHole_2.2mm_M2, symbol Mechanical:MountingHole
- removed J2: Conn_01x03, Connector_PinHeader_2.54mm:PinHeader_1x03_P2.54mm_Vertical, symbol Connector_Generic:Conn_01x03
- removed JP1: Jumper_NC_Small, Jumper:SolderJumper-2_P1.3mm_Bridged2Bar_Pad1.0x1.5mm, symbol Device:Jumper_NC_Small
- removed JP_LED1, JP_LED2: SolderJumper_3_Open, Jumper:SolderJumper-3_P1.3mm_Open_Pad1.0x1.5mm_NumberLabels, symbol Jumper:SolderJumper_3_Open
- removed LED1, LED2, LED3, LED4: SK6812MINI, locallib:LED_SK6812MINI_PLCC4_3.5x3.5mm_P1.75mm_TriangleMark, symbol LED:SK6812MINI
- removed LED_STRIP1: Conn_01x03, locallib:LED_Strip, symbol Connector_Generic:Conn_01x03
- removed Reserve_PB5, Reserve_PB6, Reserve_PB7: Conn_01x01, TestPoint:TestPoint_THTPad_D1.0mm_Drill0.5mm, symbol Connector_Generic:Conn_01x01
- removed U3: ATmega32U4-AU, Package_QFP:TQFP-44_10x10mm_P0.8mm, symbol MCU_Microchip_ATmega:ATmega32U4-AU
- added L1, L10, L11, L12, L13, L14, L15, L16, L2, L3, L4, L5, L6, L7, L8, L9: SK6812MINI-E, Jones.local:YS-SK6812MINI-E, symbol kbd:SK6812MINI-E
- added U3: ATmega32U4-AU-Dummy, Package_QFP:TQFP-44_10x10mm_P0.8mm, symbol choc_in_60:ATmega32U4-AU-Dummy
- SW_7: footprint Keebio-Parts:Kailh-PG1350-1.5u-MBK-WithKeyName -> Keebio-Parts:Kailh-PG1350-1.5u-MBK-WithKeyName-NoClickHole
- renumbered Reserve_PC6 to ReservePin1
Connections:
- net labels added: Reserve_pin
- net labels removed: resv_PB5, resv_PB6, resv_PB7, resv_PC6
- wire segments 401 -> 474
- no-connect marks 4 -> 5
Other:
- note added: "RESERVED & TEST PINS"
- note removed: "RESERVED PINS"
- note removed: "Use Left LEDs"
- note removed: "Use Right LEDs"
- moved on the sheet: J3, R8, R9, ReservePin1, U2
