File: PCB/choc_in_60.kicad_pcb (KiCad board)
At the start: 2 copper layers, 285 x 95.1 mm, 213 parts, among them J1 USB_C_Receptacle_USB2.0, J2 Conn_01x03, J3 Conn_01x02, J5 Conn_02x03_Odd_Even, U1 ATmega32U4-MU, U2 24LC64, U3 ATmega32U4-AU, Y1 16MHz

Commit message: 配線途中
Parts:
- removed H5: MountingHole, MountingHole:MountingHole_2.2mm_M2
- removed J2: Conn_01x03, Connector_PinHeader_2.54mm:PinHeader_1x03_P2.54mm_Vertical
- removed JP1: Jumper_NC_Small, Jumper:SolderJumper-2_P1.3mm_Bridged2Bar_Pad1.0x1.5mm
- removed JP_LED1, JP_LED2: SolderJumper_3_Open, Jumper:SolderJumper-3_P1.3mm_Open_Pad1.0x1.5mm_NumberLabels
- removed LED1, LED2, LED3, LED4: SK6812MINI, locallib:LED_SK6812MINI_PLCC4_3.5x3.5mm_P1.75mm_TriangleMark
- removed LED_STRIP1: Conn_01x03, locallib:LED_Strip
- removed Reserve_PB5, Reserve_PB6, Reserve_PB7: Conn_01x01, TestPoint:TestPoint_THTPad_D1.0mm_Drill0.5mm
- added L1: SK6812MINI-E, Jones.local:YS-SK6812MINI-E, B.Cu at (31.2, 31.2)
- added L10: SK6812MINI-E, Jones.local:YS-SK6812MINI-E, B.Cu at (191.9, 31.2)
- added L11: SK6812MINI-E, Jones.local:YS-SK6812MINI-E, B.Cu at (209.8, 31.2)
- added L12: SK6812MINI-E, Jones.local:YS-SK6812MINI-E, B.Cu at (227.6, 31.2)
- added L13: SK6812MINI-E, Jones.local:YS-SK6812MINI-E, B.Cu at (245.5, 31.2)
- added L14: SK6812MINI-E, Jones.local:YS-SK6812MINI-E, B.Cu at (263.3, 31.2)
- added L15: SK6812MINI-E, Jones.local:YS-SK6812MINI-E, B.Cu at (281.2, 31.2)
- added L16: SK6812MINI-E, Jones.local:YS-SK6812MINI-E, B.Cu at (299.1, 31.2)
- added L2: SK6812MINI-E, Jones.local:YS-SK6812MINI-E, B.Cu at (49.0, 31.2)
- added L3: SK6812MINI-E, Jones.local:YS-SK6812MINI-E, B.Cu at (66.9, 31.2)
- added L4: SK6812MINI-E, Jones.local:YS-SK6812MINI-E, B.Cu at (84.8, 31.2)
- added L5: SK6812MINI-E, Jones.local:YS-SK6812MINI-E, B.Cu at (102.6, 31.2)
- added L6: SK6812MINI-E, Jones.local:YS-SK6812MINI-E, B.Cu at (120.5, 31.2)
- added L7: SK6812MINI-E, Jones.local:YS-SK6812MINI-E, B.Cu at (138.3, 31.2)
- added L8: SK6812MINI-E, Jones.local:YS-SK6812MINI-E, B.Cu at (156.2, 31.2)
- added L9: SK6812MINI-E, Jones.local:YS-SK6812MINI-E, B.Cu at (174.0, 31.2)
- D1, D11, D12, D13, D14, D15, D16, D17, D18, D19, D2, D20, D21, D22, D23, D25, D26, D27, D28, D29, D3, D30, D31, D32, D33, D35, D36, D37, D38, D39, D4, D40, D41, D42, D43, D45, D46, D47, D48, D49, D5, D50, D51, D52, D53, D54, D55, D56, D57, D58, D59, D6, D60, D61, D62, D63, D64, D65, D66, D67, D68, D69, D7, D70, D71, D72, D73, D74, D75, D76, D77, D78, D79, D8, D9: moved to B.Cu
- SW_7: footprint Keebio-Parts:Kailh-PG1350-1.5u-MBK-WithKeyName -> Keebio-Parts:Kailh-PG1350-1.5u-MBK-WithKeyName-NoClickHole
- U3: value ATmega32U4-AU -> ATmega32U4-AU-Dummy
- moved D79 264.3 mm to (299.1, 107.4), turned to 180 degrees
- moved EXT_R5 259.2 mm to (304.6, 41.1), turned to 270 degrees
- moved D78 257.0 mm to (299.1, 90.4), turned to 180 degrees
- moved EXT_R6 253.2 mm to (304.6, 58.1), turned to 270 degrees
- moved EXT_R7 248.0 mm to (304.6, 75.0), turned to 270 degrees
- moved D77 247.3 mm to (299.1, 73.3), turned to 180 degrees
- moved D75 244.8 mm to (299.1, 39.4), turned to 180 degrees
- moved EXT_R8 243.5 mm to (304.6, 91.9), turned to 270 degrees
- moved EXT_R0 243.3 mm to (304.6, 38.5), turned to 90 degrees
- moved D76 242.4 mm to (299.1, 56.4), turned to 180 degrees
- moved EXT_R9 239.7 mm to (304.6, 109.0), turned to 270 degrees
- moved D74 237.1 mm to (281.2, 107.4), turned to 180 degrees
- moved EXT_R1 236.8 mm to (304.6, 55.5), turned to 90 degrees
- moved D73 233.6 mm to (281.2, 90.4), turned to 180 degrees
- moved EXT_R2 231.0 mm to (304.6, 72.4), turned to 90 degrees
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- renumbered Reserve_PC6 to ReservePin1
Connections:
- C3 pad 1: Net-(C3-Pad1) -> XTAL2
- EXT_C2 pad 1: SCK -> col2
- EXT_C4 pad 1: MOSI -> col4
- EXT_C6 pad 1: MISO -> col6
- ReservePin1 pad 1: resv_PC6 -> Reserve_pin
- SW_20 pad 1: SCK -> col2
- SW_21 pad 1: SCK -> col2
- SW_22 pad 1: SCK -> col2
- SW_23 pad 1: SCK -> col2
- SW_25 pad 1: SCK -> col2
- SW_26 pad 1: SCK -> col2
- SW_27 pad 1: SCK -> col2
- SW_28 pad 1: SCK -> col2
- SW_29 pad 1: SCK -> col2
- SW_40 pad 1: MOSI -> col4
- SW_41 pad 1: MOSI -> col4
- SW_42 pad 1: MOSI -> col4
- SW_43 pad 1: MOSI -> col4
- SW_45 pad 1: MOSI -> col4
- SW_46 pad 1: MOSI -> col4
- SW_47 pad 1: MOSI -> col4
- SW_48 pad 1: MOSI -> col4
- SW_49 pad 1: MOSI -> col4
- SW_60 pad 1: MISO -> col6
- SW_61 pad 1: MISO -> col6
- SW_62 pad 1: MISO -> col6
- SW_63 pad 1: MISO -> col6
- SW_64 pad 1: MISO -> col6
- SW_65 pad 1: MISO -> col6
- SW_66 pad 1: MISO -> col6
- SW_67 pad 1: MISO -> col6
- SW_68 pad 1: MISO -> col6
- SW_69 pad 1: MISO -> col6
- U1 pad 1: col3 -> LED
- U1 pad 12: resv_PB7 -> row1
- U1 pad 16: Net-(C3-Pad1) -> XTAL2
- U1 pad 20: row5 -> Reserve_pin
- U1 pad 21: row0 -> col4
- U1 pad 26: row7 -> col7
- U1 pad 27: row2 -> col3
- U1 pad 28: row8 -> col6
- U1 pad 29: resv_PB5 -> col2
- U1 pad 30: resv_PB6 -> row9
- U1 pad 31: resv_PC6 -> row4
- U1 pad 32: col7 -> row8
- U1 pad 36: row4 -> row3
- U1 pad 37: row9 -> row7
- U1 pad 38: row1 -> row2
- U1 pad 40: LED -> row0
- U1 pad 41: row3 -> col0
- U1 pad 8: col0 -> row5
- U3 pad 1: col3 -> LED
- U3 pad 12: resv_PB7 -> row1
- U3 pad 20: row5 -> Reserve_pin
- U3 pad 21: row0 -> col4
- U3 pad 26: row7 -> col7
- U3 pad 27: row2 -> col3
- U3 pad 28: row8 -> col6
- U3 pad 29: resv_PB5 -> col2
- U3 pad 30: resv_PB6 -> row9
- U3 pad 31: resv_PC6 -> row4
- U3 pad 32: col7 -> row8
- U3 pad 36: row4 -> row3
- U3 pad 37: row9 -> row7
- U3 pad 38: row1 -> row2
- U3 pad 40: LED -> row0
- U3 pad 41: row3 -> col0
- U3 pad 8: col0 -> row5
- Y1 pad 3: Net-(C3-Pad1) -> XTAL2
Routing:
- net GND: track 0.00 -> 319.6 mm
- net +5V: track 0.00 -> 284.7 mm
- net row3: track 0.00 -> 284.2 mm
- net row0: track 0.00 -> 280.7 mm
- net row4: track 0.00 -> 280.6 mm
- net row5: track 0.00 -> 278.7 mm
- net row8: track 0.00 -> 273.3 mm
- net row9: track 0.00 -> 270.5 mm
- net row1: track 0.00 -> 253.4 mm
- net row2: track 0.00 -> 252.1 mm
- net row7: track 0.00 -> 241.4 mm
- net row6: track 0.00 -> 241.0 mm
- net col5: track 0.00 -> 186.8 mm
- net col6: track 0.00 -> 178.3 mm
- net col7: track 0.00 -> 170.5 mm
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- removed copper zone on F.Cu, net GND
Other:
- board text added: "#Jones_mbk v.0.1 a cosmopolitan's keyboard, by @jpskenn"
- board text removed: "#Jones_mbk v.0.1, a cosmopolitan's keyboard by @jpskenn"
- board text removed: "2.25u 2u"

Commit message: 配線途中
Parts:
- moved D10 18.1 mm to (31.4, 25.1), turned to 270 degrees
- moved R1 4.40 mm to (50.2, 24.0)
- moved F1 4.40 mm to (50.9, 26.4)
- moved R2 4.16 mm to (31.4, 28.5), turned to 0 degrees
- moved R3 2.37 mm to (40.8, 34.2)
- moved R4 1.16 mm to (40.8, 31.3), turned to 0 degrees
- moved U1 0.40 mm to (43.7, 61.4)
- moved U3 0.40 mm to (43.7, 61.4)
Routing:
- net row0: track 280.7 -> 244.1 mm
- net +5V: track 284.7 -> 314.0 mm, vias 0 -> 4
- net D-: track 2.67 -> 28.0 mm
- net D+: track 2.54 -> 23.8 mm
- net col0: track 134.7 -> 116.8 mm
- net VCC: track 6.54 -> 21.5 mm, vias 0 -> 2
- net Net-(L1-Pad2): track 0.00 -> 13.5 mm, vias 0 -> 2
- net Net-(J1-PadB5): track 0.00 -> 10.8 mm, vias 0 -> 1
- net XTAL2: track 13.4 -> 5.42 mm
- net GND: track 319.6 -> 325.3 mm, vias 0 -> 1
- net XTAL1: track 9.81 -> 4.85 mm
- net Net-(J1-PadA5): track 9.55 -> 8.16 mm, vias 0 -> 1
- net Net-(D10-Pad2): track 16.1 -> 17.2 mm, vias 0 -> 1
- net Net-(D10-Pad3): track 14.9 -> 14.2 mm, vias 0 -> 1
