File: PCB/nora.sch (KiCad schematic (older format))
At the start: 231 parts, among them J1 USB_C_Receptacle_USB2.0, J2 Conn_01x04, J3 Conn_01x02, J5 Conn_02x03_Odd_Even, U1 ATmega32U4-MU, U2 24LC64, U4 Pico, Y1 16MHz

Commit message: LED光を反射するペイントを追加#32
Parts:
- L1, L10, L11, L12, L13, L14, L15, L16, L17, L18, L19, L2, L20, L21, L22, L23, L24, L25, L26, L27, L28, L29, L3, L4, L5, L6, L7, L8, L9: footprint Jones.local:YS-SK6812MINI-E -> Jones.local:YS-SK6812MINI-E_with_reflection_paint
Changed lines of the file:
@@
 F 0 "L2" H 1650 8613 51  0000 C CNN
 F 1 "SK6812MINI-E" H 1650 8678 16  0000 C CNN
-F 2 "Jones.local:YS-SK6812MINI-E" H 1650 8875 60  0001 C CNN
+F 2 "Jones.local:YS-SK6812MINI-E_with_reflection_paint" H 1650 8875 60  0001 C CNN
 F 3 "" H 1650 8875 60  0001 C CNN
 	1    1650 8875
@@
 F 0 "L1" H 1225 8613 51  0000 C CNN
 F 1 "SK6812MINI-E" H 1225 8678 16  0000 C CNN
-F 2 "Jones.local:YS-SK6812MINI-E" H 1225 8875 60  0001 C CNN
+F 2 "Jones.local:YS-SK6812MINI-E_with_reflection_paint" H 1225 8875 60  0001 C CNN
 F 3 "" H 1225 8875 60  0001 C CNN
 	1    1225 8875
@@
 F 0 "L4" H 2500 8613 51  0000 C CNN
 F 1 "SK6812MINI-E" H 2500 8678 16  0000 C CNN
-F 2 "Jones.local:YS-SK6812MINI-E" H 2500 8875 60  0001 C CNN
+F 2 "Jones.local:YS-SK6812MINI-E_with_reflection_paint" H 2500 8875 60  0001 C CNN
 F 3 "" H 2500 8875 60  0001 C CNN
 	1    2500 8875
@@
 F 0 "L3" H 2075 8613 51  0000 C CNN
 F 1 "SK6812MINI-E" H 2075 8678 16  0000 C CNN
-F 2 "Jones.local:YS-SK6812MINI-E" H 2075 8875 60  0001 C CNN
+F 2 "Jones.local:YS-SK6812MINI-E_with_reflection_paint" H 2075 8875 60  0001 C CNN
 F 3 "" H 2075 8875 60  0001 C CNN
 	1    2075 8875
@@
 F 0 "L6" H 3350 8613 51  0000 C CNN
 F 1 "SK6812MINI-E" H 3350 8678 16  0000 C CNN
-F 2 "Jones.local:YS-SK6812MINI-E" H 3350 8875 60  0001 C CNN
+F 2 "Jones.local:YS-SK6812MINI-E_with_reflection_paint" H 3350 8875 60  0001 C CNN
 F 3 "" H 3350 8875 60  0001 C CNN
 	1    3350 8875
@@
 F 0 "L5" H 2925 8613 51  0000 C CNN
 F 1 "SK6812MINI-E" H 2925 8678 16  0000 C CNN
-F 2 "Jones.local:YS-SK6812MINI-E" H 2925 8875 60  0001 C CNN
+F 2 "Jones.local:YS-SK6812MINI-E_with_reflection_paint" H 2925 8875 60  0001 C CNN
 F 3 "" H 2925 8875 60  0001 C CNN
 	1    2925 8875
@@
 F 0 "L8" H 4200 8613 51  0000 C CNN
 F 1 "SK6812MINI-E" H 4200 8678 16  0000 C CNN
-F 2 "Jones.local:YS-SK6812MINI-E" H 4200 8875 60  0001 C CNN
+F 2 "Jones.local:YS-SK6812MINI-E_with_reflection_paint" H 4200 8875 60  0001 C CNN
 F 3 "" H 4200 8875 60  0001 C CNN
 	1    4200 8875
@@
 F 0 "L7" H 3775 8613 51  0000 C CNN
 F 1 "SK6812MINI-E" H 3775 8678 16  0000 C CNN
-F 2 "Jones.local:YS-SK6812MINI-E" H 3775 8875 60  0001 C CNN
+F 2 "Jones.local:YS-SK6812MINI-E_with_reflection_paint" H 3775 8875 60  0001 C CNN
 F 3 "" H 3775 8875 60  0001 C CNN
 	1    3775 8875
@@
 F 0 "L10" H 5050 8613 51  0000 C CNN
 F 1 "SK6812MINI-E" H 5050 8678 16  0000 C CNN
-F 2 "Jones.local:YS-SK6812MINI-E" H 5050 8875 60  0001 C CNN
+F 2 "Jones.local:YS-SK6812MINI-E_with_reflection_paint" H 5050 8875 60  0001 C CNN
 F 3 "" H 5050 8875 60  0001 C CNN
 	1    5050 8875
@@
 F 0 "L9" H 4625 8613 51  0000 C CNN
 F 1 "SK6812MINI-E" H 4625 8678 16  0000 C CNN
-F 2 "Jones.local:YS-SK6812MINI-E" H 4625 8875 60  0001 C CNN
+F 2 "Jones.local:YS-SK6812MINI-E_with_reflection_paint" H 4625 8875 60  0001 C CNN
 F 3 "" H 4625 8875 60  0001 C CNN
 	1    4625 8875
@@
 F 0 "L12" H 5900 8613 51  0000 C CNN
 F 1 "SK6812MINI-E" H 5900 8678 16  0000 C CNN
-F 2 "Jones.local:YS-SK6812MINI-E" H 5900 8875 60  0001 C CNN
+F 2 "Jones.local:YS-SK6812MINI-E_with_reflection_paint" H 5900 8875 60  0001 C CNN
 F 3 "" H 5900 8875 60  0001 C CNN
 	1    5900 8875
@@
 F 0 "L11" H 5475 8613 51  0000 C CNN
 F 1 "SK6812MINI-E" H 5475 8678 16  0000 C CNN
-F 2 "Jones.local:YS-SK6812MINI-E" H 5475 8875 60  0001 C CNN
+F 2 "Jones.local:YS-SK6812MINI-E_with_reflection_paint" H 5475 8875 60  0001 C CNN
 F 3 "" H 5475 8875 60  0001 C CNN
 	1    5475 8875
@@
 F 0 "L14" H 6750 8613 51  0000 C CNN
 F 1 "SK6812MINI-E" H 6750 8678 16  0000 C CNN
-F 2 "Jones.local:YS-SK6812MINI-E" H 6750 8875 60  0001 C CNN
+F 2 "Jones.local:YS-SK6812MINI-E_with_reflection_paint" H 6750 8875 60  0001 C CNN
 F 3 "" H 6750 8875 60  0001 C CNN
 	1    6750 8875
@@
 F 0 "L13" H 6325 8613 51  0000 C CNN
 F 1 "SK6812MINI-E" H 6325 8678 16  0000 C CNN
-F 2 "Jones.local:YS-SK6812MINI-E" H 6325 8875 60  0001 C CNN
+F 2 "Jones.local:YS-SK6812MINI-E_with_reflection_paint" H 6325 8875 60  0001 C CNN
 F 3 "" H 6325 8875 60  0001 C CNN
 	1    6325 8875
@@
 F 0 "L16" H 7600 8613 51  0000 C CNN
 F 1 "SK6812MINI-E" H 7600 8678 16  0000 C CNN
-F 2 "Jones.local:YS-SK6812MINI-E" H 7600 8875 60  0001 C CNN
+F 2 "Jones.local:YS-SK6812MINI-E_with_reflection_paint" H 7600 8875 60  0001 C CNN
 F 3 "" H 7600 8875 60  0001 C CNN
 	1    7600 8875
@@
 F 0 "L15" H 7175 8613 51  0000 C CNN
 F 1 "SK6812MINI-E" H 7175 8678 16  0000 C CNN
-F 2 "Jones.local:YS-SK6812MINI-E" H 7175 8875 60  0001 C CNN
+F 2 "Jones.local:YS-SK6812MINI-E_with_reflection_paint" H 7175 8875 60  0001 C CNN
 F 3 "" H 7175 8875 60  0001 C CNN
 	1    7175 8875
@@
 F 0 "L18" H 1650 9338 51  0000 C CNN
 F 1 "SK6812MINI-E" H 1650 9403 16  0000 C CNN
-F 2 "Jones.local:YS-SK6812MINI-E" H 1650 9600 60  0001 C CNN
+F 2 "Jones.local:YS-SK6812MINI-E_with_reflection_paint" H 1650 9600 60  0001 C CNN
 F 3 "" H 1650 9600 60  0001 C CNN
 	1    1650 9600
@@
 F 0 "L17" H 1225 9338 51  0000 C CNN
 F 1 "SK6812MINI-E" H 1225 9403 16  0000 C CNN
-F 2 "Jones.local:YS-SK6812MINI-E" H 1225 9600 60  0001 C CNN
+F 2 "Jones.local:YS-SK6812MINI-E_with_reflection_paint" H 1225 9600 60  0001 C CNN
 F 3 "" H 1225 9600 60  0001 C CNN
 	1    1225 9600
@@
 F 0 "L20" H 2500 9338 51  0000 C CNN
 F 1 "SK6812MINI-E" H 2500 9403 16  0000 C CNN
-F 2 "Jones.local:YS-SK6812MINI-E" H 2500 9600 60  0001 C CNN
+F 2 "Jones.local:YS-SK6812MINI-E_with_reflection_paint" H 2500 9600 60  0001 C CNN
 F 3 "" H 2500 9600 60  0001 C CNN
 	1    2500 9600
@@
 F 0 "L19" H 2075 9338 51  0000 C CNN
 F 1 "SK6812MINI-E" H 2075 9403 16  0000 C CNN
-F 2 "Jones.local:YS-SK6812MINI-E" H 2075 9600 60  0001 C CNN
+F 2 "Jones.local:YS-SK6812MINI-E_with_reflection_paint" H 2075 9600 60  0001 C CNN
 F 3 "" H 2075 9600 60  0001 C CNN
 	1    2075 9600
@@
 F 0 "L22" H 3350 9338 51  0000 C CNN
 F 1 "SK6812MINI-E" H 3350 9403 16  0000 C CNN
-F 2 "Jones.local:YS-SK6812MINI-E" H 3350 9600 60  0001 C CNN
+F 2 "Jones.local:YS-SK6812MINI-E_with_reflection_paint" H 3350 9600 60  0001 C CNN
 F 3 "" H 3350 9600 60  0001 C CNN
 	1    3350 9600
@@
 F 0 "L21" H 2925 9338 51  0000 C CNN
 F 1 "SK6812MINI-E" H 2925 9403 16  0000 C CNN
-F 2 "Jones.local:YS-SK6812MINI-E" H 2925 9600 60  0001 C CNN
+F 2 "Jones.local:YS-SK6812MINI-E_with_reflection_paint" H 2925 9600 60  0001 C CNN
 F 3 "" H 2925 9600 60  0001 C CNN
 	1    2925 9600
@@
 F 0 "L24" H 4200 9338 51  0000 C CNN
 F 1 "SK6812MINI-E" H 4200 9403 16  0000 C CNN
-F 2 "Jones.local:YS-SK6812MINI-E" H 4200 9600 60  0001 C CNN
+F 2 "Jones.local:YS-SK6812MINI-E_with_reflection_paint" H 4200 9600 60  0001 C CNN
 F 3 "" H 4200 9600 60  0001 C CNN
 	1    4200 9600
@@
 F 0 "L23" H 3775 9338 51  0000 C CNN
 F 1 "SK6812MINI-E" H 3775 9403 16  0000 C CNN
-F 2 "Jones.local:YS-SK6812MINI-E" H 3775 9600 60  0001 C CNN
+F 2 "Jones.local:YS-SK6812MINI-E_with_reflection_paint" H 3775 9600 60  0001 C CNN
 F 3 "" H 3775 9600 60  0001 C CNN
 	1    3775 9600
@@
 F 0 "L26" H 5050 9338 51  0000 C CNN
 F 1 "SK6812MINI-E" H 5050 9403 16  0000 C CNN
-F 2 "Jones.local:YS-SK6812MINI-E" H 5050 9600 60  0001 C CNN
+F 2 "Jones.local:YS-SK6812MINI-E_with_reflection_paint" H 5050 9600 60  0001 C CNN
 F 3 "" H 5050 9600 60  0001 C CNN
 	1    5050 9600
@@
 F 0 "L25" H 4625 9338 51  0000 C CNN
 F 1 "SK6812MINI-E" H 4625 9403 16  0000 C CNN
-F 2 "Jones.local:YS-SK6812MINI-E" H 4625 9600 60  0001 C CNN
+F 2 "Jones.local:YS-SK6812MINI-E_with_reflection_paint" H 4625 9600 60  0001 C CNN
 F 3 "" H 4625 9600 60  0001 C CNN
 	1    4625 9600
@@
 F 0 "L28" H 5900 9338 51  0000 C CNN
 F 1 "SK6812MINI-E" H 5900 9403 16  0000 C CNN
-F 2 "Jones.local:YS-SK6812MINI-E" H 5900 9600 60  0001 C CNN
+F 2 "Jones.local:YS-SK6812MINI-E_with_reflection_paint" H 5900 9600 60  0001 C CNN
 F 3 "" H 5900 9600 60  0001 C CNN
 	1    5900 9600
@@
 F 0 "L27" H 5475 9338 51  0000 C CNN
 F 1 "SK6812MINI-E" H 5475 9403 16  0000 C CNN
-F 2 "Jones.local:YS-SK6812MINI-E" H 5475 9600 60  0001 C CNN
+F 2 "Jones.local:YS-SK6812MINI-E_with_reflection_paint" H 5475 9600 60  0001 C CNN
 F 3 "" H 5475 9600 60  0001 C CNN
 	1    5475 9600
@@
 F 0 "L29" H 6325 9338 51  0000 C CNN
 F 1 "SK6812MINI-E" H 6325 9403 16  0000 C CNN
-F 2 "Jones.local:YS-SK6812MINI-E" H 6325 9600 60  0001 C CNN
+F 2 "Jones.local:YS-SK6812MINI-E_with_reflection_paint" H 6325 9600 60  0001 C CNN
 F 3 "" H 6325 9600 60  0001 C CNN
 	1    6325 9600

Commit message: カーソル”上”へLED追加#35
Parts:
- added L30: SK6812MINI-E, Jones.local:YS-SK6812MINI-E_with_reflection_paint, symbol kbd:SK6812MINI-E
Connections:
- net GND: now also L30.3 (GND)
- net LED_VDD: now also L30.1 (VDD)
- net at L29.2 (DOUT): now also L30.4 (DIN)
Changed lines of the file:
@@
 $EndComp
 Wire Wire Line
-	6525 9700 6525 9800
+	6950 9700 6950 9800
 Connection ~ 1025 9375
 Wire Wire Line
@@
 Text GLabel 1025 9800 0    50   Input ~ 0
 LED_VDD
-NoConn ~ 6525 9500
+NoConn ~ 6950 9500
+Wire Wire Line
+	6525 9700 6525 9800
+Wire Wire Line
+	6525 9500 6525 9600
+Wire Wire Line
+	6525 9600 6550 9600
+Wire Wire Line
+	6550 9600 6550 9700
+Wire Wire Line
+	6550 9500 6550 9375
+$Comp
+L kbd:SK6812MINI-E L30
+U 1 1 61C12E1B
+P 6750 9600
+F 0 "L30" H 6750 9338 51  0000 C CNN
+F 1 "SK6812MINI-E" H 6750 9403 16  0000 C CNN
+F 2 "Jones.local:YS-SK6812MINI-E_with_reflection_paint" H 6750 9600 60  0001 C CNN
+F 3 "" H 6750 9600 60  0001 C CNN
+	1    6750 9600
+	-1   0    0    1
+$EndComp
+Wire Wire Line
+	6550 9375 6125 9375
+Wire Wire Line
+	6950 9800 6525 9800
+Connection ~ 6125 9375
+Connection ~ 6525 9800
 $EndSCHEMATC

Commit message: パッド強化したフットプリントに変更し、LEDを上側にもってきた
Parts:
- SW_1, SW_3, SW_4: footprint Keebio-Parts:Kailh-PG1350-1u-MBK-WithKeyName-Socket -> Keebio-Parts:Kailh-PG1350-1u-MBK-WithKeyName-Socket-ForLeftEdge2
Changed lines of the file:
@@
 F 0 "SW_3" H 1175 5535 50  0000 C CNN
 F 1 "SFT1u" H 1175 5444 50  0000 C CNN
-F 2 "Keebio-Parts:Kailh-PG1350-1u-MBK-WithKeyName-Socket" H 1175 5450 50  0001 C CNN
+F 2 "Keebio-Parts:Kailh-PG1350-1u-MBK-WithKeyName-Socket-ForLeftEdge2" H 1175 5450 50  0001 C CNN
 F 3 "~" H 1175 5450 50  0001 C CNN
 	1    1175 5250
@@
 F 0 "SW_4" H 1175 6785 50  0000 C CNN
 F 1 "LB1" H 1175 6694 50  0000 C CNN
-F 2 "Keebio-Parts:Kailh-PG1350-1u-MBK-WithKeyName-Socket" H 1175 6700 50  0001 C CNN
+F 2 "Keebio-Parts:Kailh-PG1350-1u-MBK-WithKeyName-Socket-ForLeftEdge2" H 1175 6700 50  0001 C CNN
 F 3 "~" H 1175 6700 50  0001 C CNN
 	1    1175 6500
@@
 F 0 "SW_1" H 1175 1785 50  0000 C CNN
 F 1 "ESC" H 1175 1694 50  0000 C CNN
-F 2 "Keebio-Parts:Kailh-PG1350-1u-MBK-WithKeyName-Socket" H 1175 1700 50  0001 C CNN
+F 2 "Keebio-Parts:Kailh-PG1350-1u-MBK-WithKeyName-Socket-ForLeftEdge2" H 1175 1700 50  0001 C CNN
 F 3 "~" H 1175 1700 50  0001 C CNN
 	1    1175 1500

Commit message: PICO時、EEPROMの電源をPICO-VBUSからとる#47#16
Parts:
- added J4: Conn_01x02, Connector_PinHeader_2.54mm:PinHeader_1x02_P2.54mm_Vertical, symbol Connector_Generic:Conn_01x02
Connections:
- net +5V: no longer R8.1, R9.1, U2.8 (VCC)
- net GND: now also J4.1 (Pin_1)
- net LED_VDD renamed +5V_Source
- net +5V_Source: now also R8.1, R9.1, U2.8 (VCC), J4.2 (Pin_2)
Other:
- note added: "Power Source\nfor devices"
- note removed: "I2C"
- moved on the sheet: JP3
Changed lines of the file:
@@
 L power:+5V #PWR024
 U 1 1 5F935DB7
-P 600 8875
-F 0 "#PWR024" H 600 8725 50  0001 C CNN
-F 1 "+5V" H 615 9048 50  0000 C CNN
-F 2 "" H 600 8875 50  0001 C CNN
-F 3 "" H 600 8875 50  0001 C CNN
-	1    600  8875
+P 6050 10500
+F 0 "#PWR024" H 6050 10350 50  0001 C CNN
+F 1 "+5V" H 6065 10673 50  0000 C CNN
+F 2 "" H 6050 10500 50  0001 C CNN
+F 3 "" H 6050 10500 50  0001 C CNN
+	1    6050 10500
 	1    0    0    -1
 $EndComp
@@
 	10975 9350 11100 9350
 $Comp
-L power:+5V #PWR030
-U 1 1 60CFF674
-P 10650 8550
-F 0 "#PWR030" H 10650 8400 50  0001 C CNN
-F 1 "+5V" H 10650 8690 50  0000 C CNN
-F 2 "" H 10650 8550 50  0001 C CNN
-F 3 "" H 10650 8550 50  0001 C CNN
-	1    10650 8550
-	1    0    0    -1
-$EndComp
-$Comp
-L power:+5V #PWR031
-U 1 1 60D34CB6
-P 10975 8550
-F 0 "#PWR031" H 10975 8400 50  0001 C CNN
-F 1 "+5V" H 10975 8690 50  0000 C CNN
-F 2 "" H 10975 8550 50  0001 C CNN
-F 3 "" H 10975 8550 50  0001 C CNN
-	1    10975 8550
-	1    0    0    -1
-$EndComp
-$Comp
 L Mechanical:MountingHole H1
 U 1 1 60B084C7
@@
 	8500 9175 8500 9275
 Wire Wire Line
-	8500 8575 8900 8575
-Wire Wire Line
-	8500 8475 8500 8575
-$Comp
-L power:+5V #PWR0102
-U 1 1 60AF154D
-P 8500 8475
-F 0 "#PWR0102" H 8500 8325 50  0001 C CNN
-F 1 "+5V" H 8500 8615 50  0000 C CNN
-F 2 "" H 8500 8475 50  0001 C CNN
-F 3 "" H 8500 8475 50  0001 C CNN
-	1    8500 8475
-	1    0    0    -1
-$EndComp
+	9000 8575 8900 8575
 Wire Wire Line
 	9300 9175 8900 9175
@@
 Text Notes 8400 8275 0    100  ~ 20
 EEPROM
-Text Notes 10350 8275 0    100  ~ 20
-I2C
 Text Notes 650  10175 0    100  ~ 20
 LOGO
@@
 	7400 8650 6975 8650
 Connection ~ 1425 9075
-Wire Wire Line
-	1425 9075 775  9075
 Connection ~ 1850 9075
 Wire Wire Line
@@
 	-1   0    0    1
 $EndComp
-Text GLabel 600  9275 2    50   Input ~ 0
+Text GLabel 6050 10900 2    50   Input ~ 0
 PICO_VBUS
 $Comp
@@
 L power:PWR_FLAG #FLG0102
 U 1 1 62AE90E6
-P 775 9075
-F 0 "#FLG0102" H 775 9150 50  0001 C CNN
-F 1 "PWR_FLAG" H 775 9248 50  0000 C CNN
-F 2 "" H 775 9075 50  0001 C CNN
-F 3 "~" H 775 9075 50  0001 C CNN
-	1    775  9075
+P 6375 10700
+F 0 "#FLG0102" H 6375 10775 50  0001 C CNN
+F 1 "PWR_FLAG" H 6375 10873 50  0000 C CNN
+F 2 "" H 6375 10700 50  0001 C CNN
+F 3 "~" H 6375 10700 50  0001 C CNN
+	1    6375 10700
 	1    0    0    -1
 $EndComp
-Connection ~ 775  9075
-Wire Wire Line
-	775  9075 750  9075
 $Comp
 L Jumper:SolderJumper_3_Open JP3
 U 1 1 62AEB2BC
-P 600 9075
-F 0 "JP3" V 646 9142 50  0000 L CNN
-F 1 "SolderJumper_3_Open" V 555 9142 50  0000 L CNN
-F 2 "Jumper:SolderJumper-3_P1.3mm_Open_RoundedPad1.0x1.5mm" H 600 9075 50  0001 C CNN
-F 3 "~" H 600 9075 50  0001 C CNN
-	1    600  9075
+P 6050 10700
+F 0 "JP3" V 6096 10767 50  0000 L CNN
+F 1 "SolderJumper_3_Open" V 6005 10767 50  0000 L CNN
+F 2 "Jumper:SolderJumper-3_P1.3mm_Open_RoundedPad1.0x1.5mm" H 6050 10700 50  0001 C CNN
+F 3 "~" H 6050 10700 50  0001 C CNN
+	1    6050 10700
 	0    -1   -1   0
 $EndComp
@@
 Connection ~ 6125 9375
 Connection ~ 6525 9800
+Text Notes 5150 10250 0    100  ~ 20
+Power Source\nfor devices
+Wire Wire Line
+	6200 10700 6375 10700
+Wire Wire Line
+	1025 9075 1425 9075
+Connection ~ 6375 10700
+Wire Wire Line
+	6375 10700 6625 10700
+Text GLabel 6625 10700 2    50   Input ~ 0
++5V_Source
+Text GLabel 1025 9075 0    50   Input ~ 0
++5V_Source
+Text GLabel 10575 8475 0    50   Input ~ 0
++5V_Source
+Wire Wire Line
+	10575 8475 10650 8475
+Wire Wire Line
+	10650 8475 10650 8550
+Wire Wire Line
+	10650 8475 10975 8475
+Wire Wire Line
+	10975 8475 10975 8550
+Connection ~ 10650 8475
+Text GLabel 9000 8575 2    50   Input ~ 0
++5V_Source
+$Comp
+L Connector_Generic:Conn_01x02 J4
+U 1 1 621BD6CD
+P 10600 10675
+F 0 "J4" H 10518 10350 50  0000 C CNN
+F 1 "Conn_01x02" H 10518 10441 50  0000 C CNN
+F 2 "Connector_PinHeader_2.54mm:PinHeader_1x02_P2.54mm_Vertical" H 10600 10675 50  0001 C CNN
+F 3 "~" H 10600 10675 50  0001 C CNN
+	1    10600 10675
+	-1   0    0    1
+$EndComp
+Text GLabel 10800 10575 2    50   Input ~ 0
++5V_Source
+$Comp
+L power:GND #PWR05
+U 1 1 62221C1D
+P 10800 10675
+F 0 "#PWR05" H 10800 10425 50  0001 C CNN
+F 1 "GND" H 10805 10502 50  0000 C CNN
+F 2 "" H 10800 10675 50  0001 C CNN
+F 3 "" H 10800 10675 50  0001 C CNN
+	1    10800 10675
+	1    0    0    -1
+$EndComp
 $EndSCHEMATC
