File: Plate/keyplate/keyplate.kicad_pcb (KiCad board)
At the start: 2 copper layers, 285.4 x 94.9 mm, 2 parts

Commit message: プレートの外形を基板に作成
Parts:
- removed G***: LOGO, locallib:Jones_logo_B_8.3x13.9
- moved REF** 87.6 mm to (99.6, 110.4)
Other:
- outline, holes or cut-outs redrawn
- board text removed: "#Jones_kbd Keyplate v.4.0.2, @jpskenn"
- board text removed: "JLCJLCJLCJLC"

Commit message: SWプレートにパターンを追加
Parts:
- added G***: LOGO, locallib:Nora_silk, F.Cu at (155.9, 31.3)
- added G***: LOGO, locallib:Nora_mask, F.Cu at (159.7, 31.2)
- added G***: LOGO, locallib:Nora_mask, F.Cu at (156.9, 104.2)
- added G***: LOGO, locallib:Nora_silk, F.Cu at (160.6, 104.2)
Other:
- board text added: "#Nora_kbd Switch plate v.0.1 by @jpskenn"
- board text added: "JLCJLCJLCJLC"

Commit message: Update and Change version information.#18#21
Other:
- board text added: "#Nora_kbd Switch plate DN0020 by @jpskenn"
- board text removed: "#Nora_kbd Switch plate v.0.1 by @jpskenn"
