File: Plate/keyplate/keyplate.kicad_pcb (KiCad board)
At the start: 2 copper layers, 285.4 x 94.9 mm, 5 parts

Commit message: 貼り付け箇所を描画した#6
Other:
- board text added: "* * *"
- board text added: "PICO"
- board text added: "PICO reserved area. When use PICO, place sheets below(* * *)."
- board text added: "USB"
Changed lines of the file:
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@@
   (general
     (thickness 1.6)
-    (drawings 474)
+    (drawings 557)
     (tracks 0)
     (zones 0)
@@
     (35 F.Paste user)
     (36 B.SilkS user)
-    (37 F.SilkS user)
+    (37 F.SilkS user hide)
     (38 B.Mask user)
-    (39 F.Mask user)
+    (39 F.Mask user hide)
     (40 Dwgs.User user)
     (41 Cmts.User user)
@@
     (pad 1 np_thru_hole circle (at 0 0) (size 5.3 5.3) (drill 5.3) (layers *.Cu *.Mask))
   )
+  (gr_line (start 229.75 99.75) (end 229.75 112.5) (layer B.SilkS) (width 2))
+  (gr_line (start 247.5 99.75) (end 247.5 112.5) (layer B.SilkS) (width 2))
+  (gr_line (start 29.1 25) (end 36.7 25) (layer B.SilkS) (width 0.5))
+  (gr_arc (start 36.7 23.5) (end 36.7 25) (angle -180) (layer B.SilkS) (width 0.5))
+  (gr_line (start 29.1 22) (end 36.7 22) (layer B.SilkS) (width 0.5))
+  (gr_arc (start 29.1 23.5) (end 29.1 22) (angle -180) (layer B.SilkS) (width 0.5))
+  (gr_text USB (at 32.9 23.6) (layer B.SilkS)
+    (effects (font (size 1 1) (thickness 0.15)) (justify mirror))
+  )
+  (gr_arc (start 194 28.05) (end 195 28.15) (angle -185.7441159) (layer B.SilkS) (width 0.3))
+  (gr_line (start 195 39.749415) (end 195 28.15) (layer B.SilkS) (width 0.3))
+  (gr_arc (start 194 39.75) (end 193 39.75) (angle -180.033518) (layer B.SilkS) (width 0.3))
+  (gr_line (start 192.995013 28.050588) (end 193 39.75) (layer B.SilkS) (width 0.3))
+  (gr_text "*   *   *" (at 194.25 37.4 90) (layer B.SilkS)
+    (effects (font (size 1 1) (thickness 0.15)) (justify right mirror))
+  )
+  (gr_arc (start 176.1 28.05) (end 177.1 28.15) (angle -185.7441159) (layer B.SilkS) (width 0.3))
+  (gr_line (start 177.1 39.749415) (end 177.1 28.15) (layer B.SilkS) (width 0.3))
+  (gr_arc (start 176.1 39.75) (end 175.1 39.75) (angle -180.033518) (layer B.SilkS) (width 0.3))
+  (gr_line (start 175.095013 28.050588) (end 175.1 39.75) (layer B.SilkS) (width 0.3))
+  (gr_text "*   *   *" (at 176.35 37.4 90) (layer B.SilkS)
+    (effects (font (size 1 1) (thickness 0.15)) (justify right mirror))
+  )
+  (gr_arc (start 158.2 28.05) (end 159.2 28.15) (angle -185.7441159) (layer B.SilkS) (width 0.3))
+  (gr_line (start 159.2 39.749415) (end 159.2 28.15) (layer B.SilkS) (width 0.3))
+  (gr_arc (start 158.2 39.75) (end 157.2 39.75) (angle -180.033518) (layer B.SilkS) (width 0.3))
+  (gr_line (start 157.195013 28.050588) (end 157.2 39.75) (layer B.SilkS) (width 0.3))
+  (gr_text "*   *   *" (at 158.45 37.4 90) (layer B.SilkS)
+    (effects (font (size 1 1) (thickness 0.15)) (justify right mirror))
+  )
+  (gr_arc (start 140.35 28.05) (end 141.35 28.15) (angle -185.7441159) (layer B.SilkS) (width 0.3))
+  (gr_line (start 141.35 39.749415) (end 141.35 28.15) (layer B.SilkS) (width 0.3))
+  (gr_arc (start 140.35 39.75) (end 139.35 39.75) (angle -180.033518) (layer B.SilkS) (width 0.3))
+  (gr_line (start 139.345013 28.050588) (end 139.35 39.75) (layer B.SilkS) (width 0.3))
+  (gr_text "*   *   *" (at 140.6 37.4 90) (layer B.SilkS)
+    (effects (font (size 1 1) (thickness 0.15)) (justify right mirror))
+  )
+  (gr_arc (start 122.5 39.75) (end 121.5 39.75) (angle -180.033518) (layer B.SilkS) (width 0.3))
+  (gr_line (start 121.495013 28.050588) (end 121.5 39.75) (layer B.SilkS) (width 0.3))
+  (gr_arc (start 122.5 28.05) (end 123.5 28.15) (angle -185.7441159) (layer B.SilkS) (width 0.3))
+  (gr_line (start 123.5 39.749415) (end 123.5 28.15) (layer B.SilkS) (width 0.3))
+  (gr_text "*   *   *" (at 122.75 37.4 90) (layer B.SilkS)
+    (effects (font (size 1 1) (thickness 0.15)) (justify right mirror))
+  )
+  (gr_line (start 267 112) (end 297.5 112) (layer B.SilkS) (width 4))
+  (gr_line (start 283.25 27.75) (end 283.25 108) (layer B.SilkS) (width 2))
+  (gr_line (start 265.5 27.75) (end 265.5 91) (layer B.SilkS) (width 2))
+  (gr_arc (start 184.95 49) (end 183.95 49) (angle -180.033518) (layer B.SilkS) (width 0.3))
+  (gr_line (start 183.945013 44.800588) (end 183.946482 48.950588) (layer B.SilkS) (width 0.3))
+  (gr_arc (start 184.95 44.8) (end 185.95 44.9) (angle -185.7441159) (layer B.SilkS) (width 0.3))
+  (gr_line (start 185.951469 49.05) (end 185.95 44.9) (layer B.SilkS) (width 0.3))
+  (gr_text PICO (at 185 45.1 90) (layer B.SilkS)
+    (effects (font (size 1 1) (thickness 0.15)) (justify left mirror))
+  )
+  (gr_arc (start 167.25 49) (end 166.25 49) (angle -180.033518) (layer B.SilkS) (width 0.3))
+  (gr_line (start 166.245013 44.800588) (end 166.246482 48.950588) (layer B.SilkS) (width 0.3))
+  (gr_arc (start 167.25 44.8) (end 168.25 44.9) (angle -185.7441159) (layer B.SilkS) (width 0.3))
+  (gr_line (start 168.251469 49.05) (end 168.25 44.9) (layer B.SilkS) (width 0.3))
+  (gr_text PICO (at 167.3 45.1 90) (layer B.SilkS)
+    (effects (font (size 1 1) (thickness 0.15)) (justify left mirror))
+  )
+  (gr_text PICO (at 149.3 45.1 90) (layer B.SilkS)
+    (effects (font (size 1 1) (thickness 0.15)) (justify left mirror))
+  )
+  (gr_line (start 150.251469 49.05) (end 150.25 44.9) (layer B.SilkS) (width 0.3))
+  (gr_line (start 148.245013 44.800588) (end 148.246482 48.950588) (layer B.SilkS) (width 0.3))
+  (gr_arc (start 149.25 49) (end 148.25 49) (angle -180.033518) (layer B.SilkS) (width 0.3))
+  (gr_arc (start 149.25 44.8) (end 150.25 44.9) (angle -185.7441159) (layer B.SilkS) (width 0.3))
+  (gr_line (start 185 51.75) (end 185 74.25) (layer B.SilkS) (width 2))
+  (gr_line (start 167.25 51.75) (end 167.25 74.25) (layer B.SilkS) (width 2))
+  (gr_line (start 149.25 51.75) (end 149.25 74.25) (layer B.SilkS) (width 2))
+  (gr_line (start 131.5 44.75) (end 131.5 74.25) (layer B.SilkS) (width 2))
+  (gr_line (start 203 44.75) (end 203 74.25) (layer B.SilkS) (width 2))
+  (gr_line (start 113.5 44.75) (end 113.5 74.25) (layer B.SilkS) (width 2))
+  (gr_line (start 95.75 44.75) (end 95.75 74.25) (layer B.SilkS) (width 2))
+  (gr_line (start 78 44.75) (end 78 74.25) (layer B.SilkS) (width 2))
+  (gr_line (start 60 44.75) (end 60 74.25) (layer B.SilkS) (width 2))
+  (gr_text "PICO reserved area.  When use PICO, place sheets below(* * *)." (at 158.25 23.5) (layer B.SilkS)
+    (effects (font (size 1 1) (thickness 0.15)) (justify mirror))
+  )
+  (gr_line (start 117.5 25) (end 199 25) (layer B.SilkS) (width 0.5))
+  (gr_arc (start 117.5 23.5) (end 117.5 22) (angle -180) (layer B.SilkS) (width 0.5))
+  (gr_arc (start 199 23.5) (end 199 25) (angle -180) (layer B.SilkS) (width 0.5))
+  (gr_line (start 117.5 22) (end 199 22) (layer B.SilkS) (width 0.5))
+  (gr_line (start 33.25 94) (end 33.25 108) (layer B.SilkS) (width 2))
+  (gr_line (start 96 94) (end 96 107) (layer B.SilkS) (width 2))
+  (gr_line (start 167 94) (end 167 108) (layer B.SilkS) (width 2))
+  (gr_line (start 131.5 94) (end 131.5 108) (layer B.SilkS) (width 2))
+  (gr_line (start 53.5 95) (end 53.5 107) (layer B.SilkS) (width 4))
+  (gr_line (start 76 95) (end 76 107) (layer B.SilkS) (width 4))
+  (gr_line (start 187 95) (end 187 107) (layer B.SilkS) (width 4))
+  (gr_line (start 19.25 112) (end 91.5 112) (layer B.SilkS) (width 4))
+  (gr_line (start 108.5 112) (end 195 112) (layer B.SilkS) (width 4))
+  (gr_line (start 249 95.5) (end 264 95.5) (layer B.SilkS) (width 4))
+  (gr_line (start 208.5 95.5) (end 228.5 95.5) (layer B.SilkS) (width 4))
+  (gr_line (start 231 78.5) (end 245.5 78.5) (layer B.SilkS) (width 4))
+  (gr_line (start 245.5 45.5) (end 245.5 73) (layer B.SilkS) (width 4))
+  (gr_line (start 223 45.5) (end 223 73) (layer B.SilkS) (width 4))
+  (gr_line (start 40 54.5) (end 40 75) (layer B.SilkS) (width 4))
+  (gr_line (start 18.75 44) (end 18.75 71.5) (layer B.SilkS) (width 4))
+  (gr_line (start 19 23.5) (end 23.8 23.5) (layer B.SilkS) (width 4))
+  (gr_line (start 212.5 23.5) (end 297.5 23.5) (layer B.SilkS) (width 4))
+  (gr_line (start 41.9 23.5) (end 104 23.5) (layer B.SilkS) (width 4))
   (gr_poly (pts (xy 141.4 60.3325) (xy 139.4 60.33) (xy 139.4 59.705) (xy 141.4 59.7075)) (layer F.SilkS) (width 0.1))
   (gr_poly (pts (xy 25.32 77.3525) (xy 23.32 77.35) (xy 23.32 76.725) (xy 25.32 76.7275)) (layer F.SilkS) (width 0.1))
-  (gr_poly (pts (xy 293.23 92.9525) (xy 291.23 92.95) (xy 291.23 92.325) (xy 293.23 92.3275)) (layer F.SilkS) (width 0.1))
+  (gr_poly (pts (xy 293.25 74.1525) (xy 291.25 74.15) (xy 291.25 73.525) (xy 293.25 73.5275)) (layer F.SilkS) (width 0.1))
   (gr_poly (pts (xy 293.23 60.3225) (xy 291.23 60.32) (xy 291.23 59.695) (xy 293.23 59.6975)) (layer F.SilkS) (width 0.1))
   (gr_poly (pts (xy 275.36 43.3425) (xy 273.36 43.34) (xy 273.36 42.715) (xy 275.36 42.7175)) (layer F.SilkS) (width 0.1))
   (gr_poly (pts (xy 199.44 94.3325) (xy 197.44 94.33) (xy 197.44 93.705) (xy 199.44 93.7075)) (layer F.SilkS) (width 0.1))
-  (gr_text JLCJLCJLCJLC (at 22.3 113.2) (layer B.SilkS)
+  (gr_text JLCJLCJLCJLC (at 24.5 93.5) (layer B.SilkS)
     (effects (font (size 1 1) (thickness 0.15)) (justify mirror))
   )
-  (gr_text "#Nora_kbd Switch plate DN0020\nby @jpskenn" (at 299.4 112) (layer B.SilkS)
-    (effects (font (size 1.4 1.4) (thickness 0.16)) (justify left mirror))
+  (gr_text "#Nora_kbd Switch plate DN0020 by @jpskenn" (at 66.85 42.35) (layer B.SilkS)
+    (effects (font (size 1.3 1.3) (thickness 0.15)) (justify left mirror))
   )
   (gr_line (start 49.086057 91.732274) (end 17.346366 91.732274) (layer Edge.Cuts) (width 0.2))

Commit message: イラストパターン更新#8 ネジの上のスイッチ指標修正#5
Parts:
- removed the G*** at (155.9, 31.3)
- removed the G*** at (159.7, 31.2)
- removed the G*** at (156.9, 104.2)
- removed the G*** at (160.6, 104.2)
- added G***: LOGO, locallib:Nora_mask_DN0020, F.Cu at (159.1, 66.3)
- added G***: LOGO, locallib:Nora_silk_DN0020, F.Cu at (159.1, 66.3)
Other:
- board text added: "PICO reserved area. When use PICO, place sheets below " * * * "."
- board text removed: "PICO reserved area. When use PICO, place sheets below(* * *)."
