File: Plate/keyplate/keyplate.kicad_pcb (KiCad board)
At the start: 2 copper layers, 285.4 x 94.9 mm, 3 parts

Commit message: プレート作成
Parts:
- removed the G*** at (159.1, 66.3) (x2)
- added G***: LOGO, locallib:Nora_mask_DN0030, F.Cu at (158.6, 62.9)
- added G***: LOGO, locallib:Nora_silk_DN0030, F.Cu at (165.8, 63.0)
- added REF**: Nora_keyplate_DN0030, locallib:Nora_keyplate_DN0030, F.Cu at (53.4, 44.9)
- moved REF** 5.57 mm to (103.2, 106.1)
Other:
- outline, holes or cut-outs redrawn
- board text added: "#Nora_kbd Switch plate DN0030 by @jpskenn"
- board text removed: "#Nora_kbd Switch plate DN0020 by @jpskenn"

Commit message: 1800のファイルを元に戻す
Parts:
- removed the G*** at (158.6, 62.9)
- removed the G*** at (165.8, 63.0)
- removed the REF** at (53.4, 44.9)
- added G***: LOGO, locallib:Nora_mask_DN0020, F.Cu at (159.1, 66.3)
- added G***: LOGO, locallib:Nora_silk_DN0020, F.Cu at (159.1, 66.3)
- moved REF** 5.57 mm to (99.6, 110.4)
Other:
- outline, holes or cut-outs redrawn
- board text added: "#Nora_kbd Switch plate DN0020 by @jpskenn"
- board text removed: "#Nora_kbd Switch plate DN0030 by @jpskenn"
