File: PCB_FW/nora.kicad_pcb (KiCad board)
At the start: 2 copper layers, 285 x 95.1 mm, 277 parts, among them J1 USB_C_Receptacle_USB2.0, J2 Conn_01x04, J3 Conn_01x02, J4 Conn_01x02, J5 Conn_02x03_Odd_Even, U1 ATmega32U4-MU, U2 24LC64, U4 Pico, Y1 16MHz

Commit message: スピーカーを追加 #54
Parts:
- added D99: D_Small, locallib:D_SOD-123-Pretty_No_Reference, B.Cu at (281.8, 101.7)
- added LS1: Speaker, Buzzer_Beeper:Buzzer_Murata_PKMCS0909E4000-R1, B.Cu at (290.2, 101.8)
- added R7: 1k, Resistor_SMD:R_0805_2012Metric_Pad1.20x1.40mm_HandSolder, B.Cu at (278.0, 102.0)
- moved Ext_PC6 5.49 mm to (58.7, 103.0)
- moved EXT_R9 1.20 mm to (263.4, 112.4)
Routing:
- net Reserve_pin: track 4.90 -> 241.2 mm, vias 0 -> 1
- net Net-(D99-Pad1): track 0.00 -> 8.62 mm
- net col1: track 279.3 -> 279.9 mm
- net col6: track 433.9 -> 434.5 mm
- net GND: vias 117 -> 115

Commit message: 基板おもて側にスイッチの軸形状を模したシルクを追加#57
Parts:
- removed the REF** at (205.9, 39.3)
- removed the REF** at (116.7, 39.3)
- removed the REF** at (201.8, 106.0)
- removed the REF** at (295.3, 90.3)
- removed the REF** at (268.6, 56.3)
- removed the REF** at (143.3, 73.1)
- added REF**: ICON_Screw_Small, Jones.local:ICON_Screw_Small, F.Cu at (207.4, 43.0)
- added REF**: ICON_Screw_Small, Jones.local:ICON_Screw_Small, F.Cu at (118.2, 43.0)
- added REF**: ICON_Screw_Small, Jones.local:ICON_Screw_Small, F.Cu at (202.8, 111.0)
- added REF**: ICON_Screw_Small, Jones.local:ICON_Screw_Small, F.Cu at (296.6, 94.0)
- added REF**: ICON_Screw_Small, Jones.local:ICON_Screw_Small, F.Cu at (269.8, 60.0)
- added REF**: ICON_Screw_Small, Jones.local:ICON_Screw_Small, F.Cu at (144.6, 77.2)
- moved REF** 4.59 mm to (29.0, 94.0)
- moved REF** 4.05 mm to (100.0, 111.2)
- moved REF** 0.67 mm to (150.8, 75.4)

Commit message: 手直ししたロゴを基板に適用
Parts:
- moved G*** 3.00 mm to (174.0, 68.8)
Other:
- board text added: "#Nora_kbd Fearless Wings DN0030 by @jpskenn"
- board text added: "https://git.io/nora_kbd"
- board text removed: "#Nora_kbd DN0030 by @jpskenn, https://git.io/nora_kbd"
