File: PCB_FW/nora.kicad_sch (KiCad schematic)
At the start: 270 parts, among them J1 USB_C_Receptacle_USB2.0, J2 Conn_01x04, J3 Conn_01x02, J4 Conn_01x02, J5 Conn_02x03_Odd_Even, U1 ATmega32U4-MU, U2 24LC64, U4 Pico, Y1 16MHz

Commit message: WIP 中央キーのLEDスキップジャンパを追加
Parts:
- removed JP4: SolderJumper_3_Open, Jumper:SolderJumper-3_P1.3mm_Open_RoundedPad1.0x1.5mm, symbol Jumper:SolderJumper_3_Open
- added JP4, JP5, JP6, JP7, JP8: SolderJumper_2_Open, Jumper:SolderJumper-2_P1.3mm_Open_RoundedPad1.0x1.5mm, symbol Jumper:SolderJumper_2_Open
Connections:
- net LEDtoR2 is gone; now on an unnamed net: L17.4 (DIN)
- net Skip_R2C: now reaches L24.2 (DOUT), L25.4 (DIN)
- net Skip_R2C: now also JP5.2 (B)
- net at L23.2 (DOUT), L24.4 (DIN): now also JP5.1 (A)
- net Skip_R3C: now reaches L39.2 (DOUT), L40.4 (DIN)
- net Skip_R3C: now also JP6.2 (B)
- net at L38.2 (DOUT), L39.4 (DIN): now also JP6.1 (A)
- net at L53.2 (DOUT), L54.4 (DIN): now also JP7.1 (A)
- net Skip_R4C: now reaches L55.2 (DOUT), L56.4 (DIN)
- net Skip_R4C: now also JP7.2 (B)
- net at L7.2 (DOUT), L8.4 (DIN): now also JP4.1 (A)
- net Skip_R1C: now reaches L10.4 (DIN), L9.2 (DOUT)
- net Skip_R1C: now also JP4.2 (B)
- net at L66.2 (DOUT), L67.4 (DIN): now also JP8.1 (A)
- net Skip_R5C: now reaches L67.2 (DOUT), L68.4 (DIN)
- net Skip_R5C: now also JP8.2 (B)
- net LEDtoR5: no longer names the net of L62.2 (DOUT), L63.4 (DIN)
- net RE1_S1 renamed col4
Other:
- note added: "R2: Rright to Left"
- note added: "R4: Rright to Left"
- moved on the sheet: D99, L1, L10, L11, L12, L13, L14, L15, L16, L17, L18, L19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
