File: PCB_FW/nora.kicad_sch (KiCad schematic)
At the start: 275 parts, among them J1 USB_C_Receptacle_USB2.0, J2 Conn_01x04, J3 Conn_01x02, J4 Conn_01x02, J5 Conn_02x03_Odd_Even, U1 ATmega32U4-MU, U2 24LC64, U4 Pico, Y1 16MHz

Commit message: 取り付けないLEDに枠を追加 #88
Parts:
- L24, L38, L39, L40, L54, L55, L67, L8, L9: footprint Jones.local:YS-SK6812MINI-E_large_hole_with_small_pad -> Jones.local:YS-SK6812MINI-E_large_hole_with_small_pad_reserved
Changed lines of the file:
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@@
       (effects (font (size 0.4064 0.4064)))
     )
-    (property "Footprint" "Jones.local:YS-SK6812MINI-E_large_hole_with_small_pad" (id 2) (at 126.365 177.8 0)
+    (property "Footprint" "Jones.local:YS-SK6812MINI-E_large_hole_with_small_pad_reserved" (id 2) (at 126.365 177.8 0)
       (effects (font (size 1.524 1.524)) hide)
     )
@@
       (effects (font (size 0.4064 0.4064)))
     )
-    (property "Footprint" "Jones.local:YS-SK6812MINI-E_large_hole_with_small_pad" (id 2) (at 146.685 194.945 0)
+    (property "Footprint" "Jones.local:YS-SK6812MINI-E_large_hole_with_small_pad_reserved" (id 2) (at 146.685 194.945 0)
       (effects (font (size 1.524 1.524)) hide)
     )
@@
       (effects (font (size 0.4064 0.4064)))
     )
-    (property "Footprint" "Jones.local:YS-SK6812MINI-E_large_hole_with_small_pad" (id 2) (at 117.475 194.945 0)
+    (property "Footprint" "Jones.local:YS-SK6812MINI-E_large_hole_with_small_pad_reserved" (id 2) (at 117.475 194.945 0)
       (effects (font (size 1.524 1.524)) hide)
     )
@@
       (effects (font (size 0.4064 0.4064)))
     )
-    (property "Footprint" "Jones.local:YS-SK6812MINI-E_large_hole_with_small_pad" (id 2) (at 161.925 194.945 0)
+    (property "Footprint" "Jones.local:YS-SK6812MINI-E_large_hole_with_small_pad_reserved" (id 2) (at 161.925 194.945 0)
       (effects (font (size 1.524 1.524)) hide)
     )
@@
       (effects (font (size 0.4064 0.4064)))
     )
-    (property "Footprint" "Jones.local:YS-SK6812MINI-E_large_hole_with_small_pad" (id 2) (at 126.365 212.09 0)
+    (property "Footprint" "Jones.local:YS-SK6812MINI-E_large_hole_with_small_pad_reserved" (id 2) (at 126.365 212.09 0)
       (effects (font (size 1.524 1.524)) hide)
     )
@@
       (effects (font (size 0.4064 0.4064)))
     )
-    (property "Footprint" "Jones.local:YS-SK6812MINI-E_large_hole_with_small_pad" (id 2) (at 137.16 212.09 0)
+    (property "Footprint" "Jones.local:YS-SK6812MINI-E_large_hole_with_small_pad_reserved" (id 2) (at 137.16 212.09 0)
       (effects (font (size 1.524 1.524)) hide)
     )
@@
       (effects (font (size 0.4064 0.4064)))
     )
-    (property "Footprint" "Jones.local:YS-SK6812MINI-E_large_hole_with_small_pad" (id 2) (at 126.365 160.655 0)
+    (property "Footprint" "Jones.local:YS-SK6812MINI-E_large_hole_with_small_pad_reserved" (id 2) (at 126.365 160.655 0)
       (effects (font (size 1.524 1.524)) hide)
     )
@@
       (effects (font (size 0.4064 0.4064)))
     )
-    (property "Footprint" "Jones.local:YS-SK6812MINI-E_large_hole_with_small_pad" (id 2) (at 137.16 160.655 0)
+    (property "Footprint" "Jones.local:YS-SK6812MINI-E_large_hole_with_small_pad_reserved" (id 2) (at 137.16 160.655 0)
       (effects (font (size 1.524 1.524)) hide)
     )
@@
       (effects (font (size 0.4064 0.4064)))
     )
-    (property "Footprint" "Jones.local:YS-SK6812MINI-E_large_hole_with_small_pad" (id 2) (at 93.98 229.235 0)
+    (property "Footprint" "Jones.local:YS-SK6812MINI-E_large_hole_with_small_pad_reserved" (id 2) (at 93.98 229.235 0)
       (effects (font (size 1.524 1.524)) hide)
     )
@@
     )
     (path "/00000000-0000-0000-0000-00006283801f"
-      (reference "L8") (unit 1) (value "SK6812MINI-E") (footprint "Jones.local:YS-SK6812MINI-E_large_hole_with_small_pad")
+      (reference "L8") (unit 1) (value "SK6812MINI-E") (footprint "Jones.local:YS-SK6812MINI-E_large_hole_with_small_pad_reserved")
     )
     (path "/00000000-0000-0000-0000-000062868c1b"
-      (reference "L9") (unit 1) (value "SK6812MINI-E") (footprint "Jones.local:YS-SK6812MINI-E_large_hole_with_small_pad")
+      (reference "L9") (unit 1) (value "SK6812MINI-E") (footprint "Jones.local:YS-SK6812MINI-E_large_hole_with_small_pad_reserved")
     )
     (path "/00000000-0000-0000-0000-000062868c13"
@@
     )
     (path "/00000000-0000-0000-0000-0000620bf6c1"
-      (reference "L24") (unit 1) (value "SK6812MINI-E") (footprint "Jones.local:YS-SK6812MINI-E_large_hole_with_small_pad")
+      (reference "L24") (unit 1) (value "SK6812MINI-E") (footprint "Jones.local:YS-SK6812MINI-E_large_hole_with_small_pad_reserved")
     )
     (path "/00000000-0000-0000-0000-0000620bf6df"
@@
     )
     (path "/00000000-0000-0000-0000-0000622055d0"
-      (reference "L38") (unit 1) (value "SK6812MINI-E") (footprint "Jones.local:YS-SK6812MINI-E_large_hole_with_small_pad")
+      (reference "L38") (unit 1) (value "SK6812MINI-E") (footprint "Jones.local:YS-SK6812MINI-E_large_hole_with_small_pad_reserved")
     )
     (path "/00000000-0000-0000-0000-0000622055c8"
-      (reference "L39") (unit 1) (value "SK6812MINI-E") (footprint "Jones.local:YS-SK6812MINI-E_large_hole_with_small_pad")
+      (reference "L39") (unit 1) (value "SK6812MINI-E") (footprint "Jones.local:YS-SK6812MINI-E_large_hole_with_small_pad_reserved")
     )
     (path "/00000000-0000-0000-0000-0000622055e6"
-      (reference "L40") (unit 1) (value "SK6812MINI-E") (footprint "Jones.local:YS-SK6812MINI-E_large_hole_with_small_pad")
+      (reference "L40") (unit 1) (value "SK6812MINI-E") (footprint "Jones.local:YS-SK6812MINI-E_large_hole_with_small_pad_reserved")
     )
     (path "/00000000-0000-0000-0000-0000622055de"
@@
     )
     (path "/00000000-0000-0000-0000-000062678561"
-      (reference "L54") (unit 1) (value "SK6812MINI-E") (footprint "Jones.local:YS-SK6812MINI-E_large_hole_with_small_pad")
+      (reference "L54") (unit 1) (value "SK6812MINI-E") (footprint "Jones.local:YS-SK6812MINI-E_large_hole_with_small_pad_reserved")
     )
     (path "/00000000-0000-0000-0000-00006267857f"
-      (reference "L55") (unit 1) (value "SK6812MINI-E") (footprint "Jones.local:YS-SK6812MINI-E_large_hole_with_small_pad")
+      (reference "L55") (unit 1) (value "SK6812MINI-E") (footprint "Jones.local:YS-SK6812MINI-E_large_hole_with_small_pad_reserved")
     )
     (path "/00000000-0000-0000-0000-000062678577"
@@
     )
     (path "/00000000-0000-0000-0000-0000628c5fd2"
-      (reference "L67") (unit 1) (value "SK6812MINI-E") (footprint "Jones.local:YS-SK6812MINI-E_large_hole_with_small_pad")
+      (reference "L67") (unit 1) (value "SK6812MINI-E") (footprint "Jones.local:YS-SK6812MINI-E_large_hole_with_small_pad_reserved")
     )
     (path "/00000000-0000-0000-0000-0000628c5fca"

Commit message: FW+REで取り付けないソケットをわかりやすく #87
Parts:
- SW_37, SW_47: footprint Keebio-Parts:Kailh-PG1350-1u-MBK-WithKeyName-Socket-1.8mm-hole-reflection -> Keebio-Parts:Kailh-PG1350-1u-MBK-WithKeyName-Socket-1.8mm-hole-reflection-half-paint
Changed lines of the file:
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@@
     (property "Reference" "SW_37" (id 0) (at 145.415 74.041 0))
     (property "Value" ";:" (id 1) (at 145.415 76.3524 0))
-    (property "Footprint" "Keebio-Parts:Kailh-PG1350-1u-MBK-WithKeyName-Socket-1.8mm-hole-reflection" (id 2) (at 145.415 76.2 0)
+    (property "Footprint" "Keebio-Parts:Kailh-PG1350-1u-MBK-WithKeyName-Socket-1.8mm-hole-reflection-half-paint" (id 2) (at 145.415 76.2 0)
       (effects (font (size 1.27 1.27)) hide)
     )
@@
     (property "Reference" "SW_47" (id 0) (at 178.435 74.041 0))
     (property "Value" "'\"" (id 1) (at 178.435 76.3524 0))
-    (property "Footprint" "Keebio-Parts:Kailh-PG1350-1u-MBK-WithKeyName-Socket-1.8mm-hole-reflection" (id 2) (at 178.435 76.2 0)
+    (property "Footprint" "Keebio-Parts:Kailh-PG1350-1u-MBK-WithKeyName-Socket-1.8mm-hole-reflection-half-paint" (id 2) (at 178.435 76.2 0)
       (effects (font (size 1.27 1.27)) hide)
     )
@@
     )
     (path "/00000000-0000-0000-0000-000061ce966c"
-      (reference "SW_37") (unit 1) (value ";:") (footprint "Keebio-Parts:Kailh-PG1350-1u-MBK-WithKeyName-Socket-1.8mm-hole-reflection")
+      (reference "SW_37") (unit 1) (value ";:") (footprint "Keebio-Parts:Kailh-PG1350-1u-MBK-WithKeyName-Socket-1.8mm-hole-reflection-half-paint")
     )
     (path "/cc1d72d3-c085-42d5-b51a-f25583124fcb"
@@
     )
     (path "/00000000-0000-0000-0000-000061d01276"
-      (reference "SW_47") (unit 1) (value "'\"") (footprint "Keebio-Parts:Kailh-PG1350-1u-MBK-WithKeyName-Socket-1.8mm-hole-reflection")
+      (reference "SW_47") (unit 1) (value "'\"") (footprint "Keebio-Parts:Kailh-PG1350-1u-MBK-WithKeyName-Socket-1.8mm-hole-reflection-half-paint")
     )
     (path "/00000000-0000-0000-0000-000061d0128e"
