File: Plate_FW/keyplate/keyplate.kicad_pcb (KiCad board)
At the start: 2 copper layers, 285.4 x 94.9 mm, 4 parts

Commit message: SplitのSWプレートを作成
Parts:
- removed the G*** at (158.6, 62.9)
- removed the G*** at (165.8, 63.0)
- removed the REF** at (53.4, 44.9)
- added G***: LOGO, locallib:Nora_mask_DN0031, F.Cu at (150.3, 63.6)
- added G***: LOGO, locallib:Nora_silk_DN0031, F.Cu at (157.5, 63.6)
- moved REF** 4.49 mm to (99.0, 107.6)
Other:
- outline, holes or cut-outs redrawn
- net class Default removed
- board text added: "#Nora_kbd Switch plate DN0031 Split by @jpskenn"
- board text added: "PICO reserved area"
- board text removed: "#Nora_kbd Switch plate DN0030 by @jpskenn"
- board text removed: "* * *"
- board text removed: "PICO"
- board text removed: "PICO reserved area. When use PICO, place sheets below " * * * "."
