File: Plate_FW/keyplate/keyplate.kicad_pcb (KiCad board)
At the start: 2 copper layers, 285.4 x 94.9 mm, 3 parts

Commit message: バージョン更新 #120
Other:
- board text added: "#Nora_kbd Switch plate DN0032 Split by @jpskenn"
- board text removed: "#Nora_kbd Switch plate DN0031 Split by @jpskenn"
Changed lines of the file:
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@@
     (effects (font (size 1 1) (thickness 0.15)) (justify mirror))
   )
-  (gr_text "#Nora_kbd Switch plate DN0031 Split by @jpskenn" (at 95 73.6) (layer "B.SilkS")
+  (gr_text "#Nora_kbd Switch plate DN0032 Split by @jpskenn" (at 95 73.6) (layer "B.SilkS")
     (effects (font (size 1.3 1.3) (thickness 0.15)) (justify left mirror))
   )

Commit message: プレート名称変更 #134
Other:
- board text added: "#Nora_kbd Switch plate DN0032 FW by @jpskenn"
- board text removed: "#Nora_kbd Switch plate DN0032 Split by @jpskenn"
Changed lines of the file:
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@@
     (effects (font (size 1 1) (thickness 0.15)) (justify mirror))
   )
-  (gr_text "#Nora_kbd Switch plate DN0032 Split by @jpskenn" (at 95 73.6) (layer "B.SilkS")
+  (gr_text "#Nora_kbd Switch plate DN0032 FW by @jpskenn" (at 95 73.6) (layer "B.SilkS")
     (effects (font (size 1.3 1.3) (thickness 0.15)) (justify left mirror))
   )

Commit message: プレート類のガーバーファイル準備
Other:
- board text added: "#Nora_kbd Switch plate for FW, DN0032 by @jpskenn"
- board text removed: "#Nora_kbd Switch plate DN0032 FW by @jpskenn"
Changed lines of the file:
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@@
   (gr_line (start 18.026553 41.009719) (end 18.026553 68.509719) (layer "B.SilkS") (width 4))
   (gr_line (start 27.876553 22.259719) (end 36.976553 22.259719) (layer "B.SilkS") (width 0.5))
+  (gr_line (start 59.4 48.15) (end 59.4 65.65) (layer "B.SilkS") (width 2))
   (gr_line (start 169.5 94) (end 169.5 101.5) (layer "B.SilkS") (width 4))
   (gr_line (start 174 27.25) (end 174 34.75) (layer "B.SilkS") (width 4))
@@
   (gr_line (start 146 94) (end 146 101.5) (layer "B.SilkS") (width 4))
   (gr_arc (start 145.000588 40.398251) (mid 144.107541 39.444659) (end 145.1 38.595013) (layer "B.SilkS") (width 0.3))
+  (gr_line (start 130.8 48.15) (end 130.8 65.65) (layer "B.SilkS") (width 2))
   (gr_line (start 260.5 106.5) (end 294.5 106.5) (layer "B.SilkS") (width 10))
   (gr_line (start 168.555229 40.404927) (end 182.087533 40.4) (layer "B.SilkS") (width 0.3))
@@
   (gr_line (start 191 91.75) (end 191 99.25) (layer "B.SilkS") (width 4))
   (gr_line (start 183.441273 41.75374) (end 183.449707 43.15) (layer "B.SilkS") (width 0.3))
-  (gr_line (start 238 48) (end 238 65.5) (layer "B.SilkS") (width 2))
+  (gr_line (start 238 48.15) (end 238 65.65) (layer "B.SilkS") (width 2))
   (gr_line (start 116.776553 19.259719) (end 194.9 19.259719) (layer "B.SilkS") (width 0.5))
   (gr_line (start 107.846553 109.379719) (end 252 109.5) (layer "B.SilkS") (width 4))
-  (gr_line (start 77.276553 48) (end 77.276553 65.5) (layer "B.SilkS") (width 2))
-  (gr_line (start 95.25 48) (end 95.25 65.5) (layer "B.SilkS") (width 2))
-  (gr_line (start 113 48) (end 113 65.5) (layer "B.SilkS") (width 2))
+  (gr_line (start 77.276553 48.15) (end 77.276553 65.65) (layer "B.SilkS") (width 2))
+  (gr_line (start 95.25 48.15) (end 95.25 65.65) (layer "B.SilkS") (width 2))
+  (gr_line (start 113 48.15) (end 113 65.65) (layer "B.SilkS") (width 2))
   (gr_line (start 116.776553 22.259719) (end 194.9 22.259719) (layer "B.SilkS") (width 0.5))
+  (gr_line (start 255.9 48.15) (end 255.9 65.65) (layer "B.SilkS") (width 2))
   (gr_line (start 185.449707 43.149415) (end 185.44626 41.753731) (layer "B.SilkS") (width 0.3))
-  (gr_line (start 202.25 48) (end 202.25 65.5) (layer "B.SilkS") (width 2))
+  (gr_line (start 202.25 48.15) (end 202.25 65.65) (layer "B.SilkS") (width 2))
   (gr_line (start 39.276553 51.509719) (end 39.276553 72.009719) (layer "B.SilkS") (width 4))
   (gr_line (start 186.8 40.399991) (end 195.450297 40.40001) (layer "B.SilkS") (width 0.3))
+  (gr_line (start 184.3 48.15) (end 184.3 65.65) (layer "B.SilkS") (width 2))
   (gr_line (start 174 78.75) (end 174 86.25) (layer "B.SilkS") (width 4))
   (gr_line (start 42.25 20.759719) (end 103.526553 20.759719) (layer "B.SilkS") (width 4))
@@
   (gr_arc (start 27.876553 22.259719) (mid 26.376553 20.759719) (end 27.876553 19.259719) (layer "B.SilkS") (width 0.5))
   (gr_line (start 297.026553 41.009719) (end 297.026553 69) (layer "B.SilkS") (width 4))
-  (gr_line (start 220.25 48) (end 220.25 65.5) (layer "B.SilkS") (width 2))
+  (gr_line (start 220.25 48.15) (end 220.25 65.65) (layer "B.SilkS") (width 2))
   (gr_line (start 57.5 92) (end 18 92) (layer "B.SilkS") (width 4))
   (gr_arc (start 195.499124 38.6) (mid 196.4 39.525104) (end 195.450297 40.40001) (layer "B.SilkS") (width 0.3))
@@
     (effects (font (size 1 1) (thickness 0.15)) (justify mirror))
   )
-  (gr_text "#Nora_kbd Switch plate DN0032 FW by @jpskenn" (at 95 73.6) (layer "B.SilkS")
+  (gr_text "#Nora_kbd Switch plate for FW, DN0032 by @jpskenn" (at 95 73.6) (layer "B.SilkS")
     (effects (font (size 1.3 1.3) (thickness 0.15)) (justify left mirror))
   )

Commit message: スイッチプレート穴サイズ、横14.2→14ｍｍに変更
Other:
- outline, holes or cut-outs redrawn
- board text added: "#Nora_kbd Switch plate for FW, DN0032(2) by @jpskenn"
- board text removed: "#Nora_kbd Switch plate for FW, DN0032 by @jpskenn"
