File: Plate_FW_RE/keyplate/keyplate.kicad_pcb (KiCad board)
At the start: 2 copper layers, 285.4 x 94.9 mm, 3 parts

Commit message: バージョン更新 #120
Other:
- board text added: "#Nora_kbd Switch plate DN0032 Split w/RE by @jpskenn"
- board text removed: "#Nora_kbd Switch plate DN0031 Split w/RE by @jpskenn"
Changed lines of the file:
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@@
     (effects (font (size 1 1) (thickness 0.15)) (justify mirror))
   )
-  (gr_text "#Nora_kbd Switch plate DN0031 Split w/RE by @jpskenn" (at 99 73.5) (layer "B.SilkS")
+  (gr_text "#Nora_kbd Switch plate DN0032 Split w/RE by @jpskenn" (at 99 73.5) (layer "B.SilkS")
     (effects (font (size 1.3 1.3) (thickness 0.15)) (justify left mirror))
   )

Commit message: プレート名称変更 #134
Other:
- board text added: "#Nora_kbd Switch plate DN0032 RE by @jpskenn"
- board text removed: "#Nora_kbd Switch plate DN0032 Split w/RE by @jpskenn"
Changed lines of the file:
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@@
     (effects (font (size 1 1) (thickness 0.15)) (justify mirror))
   )
-  (gr_text "#Nora_kbd Switch plate DN0032 Split w/RE by @jpskenn" (at 99 73.5) (layer "B.SilkS")
+  (gr_text "#Nora_kbd Switch plate DN0032 RE by @jpskenn" (at 99 73.5) (layer "B.SilkS")
     (effects (font (size 1.3 1.3) (thickness 0.15)) (justify left mirror))
   )
