File: Plate_FW_RE/keyplate/keyplate.kicad_pcb (KiCad board)
At the start: 2 copper layers, 285.4 x 94.9 mm, 3 parts

Commit message: プレート類のガーバーファイル準備
Other:
- board text added: "#Nora_kbd Switch plate for RE, DN0032 by @jpskenn"
- board text removed: "#Nora_kbd Switch plate DN0032 RE by @jpskenn"
Changed lines of the file:
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@@
   (gr_line (start 133.5 59) (end 133.5 71.5) (layer "B.SilkS") (width 4))
   (gr_line (start 145.000588 40.398251) (end 146.949583 40.401749) (layer "B.SilkS") (width 0.3))
-  (gr_line (start 101.7 92.7) (end 101.7 100.2) (layer "B.SilkS") (width 4))
+  (gr_line (start 101.7 92.75) (end 101.7 100.25) (layer "B.SilkS") (width 4))
   (gr_line (start 173.8 27.2) (end 173.8 34.7) (layer "B.SilkS") (width 4))
   (gr_arc (start 194.9 19.259719) (mid 196.4 20.759719) (end 194.9 22.259719) (layer "B.SilkS") (width 0.5))
@@
   (gr_line (start 275.776553 51.009719) (end 275.776553 72.009719) (layer "B.SilkS") (width 4))
   (gr_line (start 151 50) (end 164 50) (layer "B.SilkS") (width 4))
-  (gr_line (start 255.786724 48.5) (end 255.8 65.5) (layer "B.SilkS") (width 2))
+  (gr_line (start 255.786724 48.4) (end 255.8 65.4) (layer "B.SilkS") (width 2))
   (gr_arc (start 185.44626 41.753731) (mid 185.842762 40.796493) (end 186.8 40.399991) (layer "B.SilkS") (width 0.3))
   (gr_line (start 21.096553 106.379719) (end 55.146553 106.379719) (layer "B.SilkS") (width 10))
@@
   (gr_line (start 18.026553 41.009719) (end 18.026553 68.509719) (layer "B.SilkS") (width 4))
   (gr_line (start 27.876553 22.259719) (end 36.976553 22.259719) (layer "B.SilkS") (width 0.5))
-  (gr_line (start 213.1 92.7) (end 213.1 100.2) (layer "B.SilkS") (width 4))
+  (gr_line (start 213.1 92.75) (end 213.1 100.25) (layer "B.SilkS") (width 4))
   (gr_arc (start 116.776553 22.259719) (mid 115.276553 20.759719) (end 116.776553 19.259719) (layer "B.SilkS") (width 0.5))
   (gr_arc (start 185.449707 43.149415) (mid 184.45 44.15) (end 183.449707 43.15) (layer "B.SilkS") (width 0.3))
-  (gr_line (start 238 48.5) (end 238 65.5) (layer "B.SilkS") (width 2))
+  (gr_line (start 238 48.4) (end 238 65.4) (layer "B.SilkS") (width 2))
   (gr_arc (start 182.087533 40.4) (mid 183.044771 40.796502) (end 183.441273 41.75374) (layer "B.SilkS") (width 0.3))
   (gr_line (start 273.525 40.6) (end 278.275 40.6) (layer "B.SilkS") (width 2))
@@
   (gr_line (start 107.846553 109.379719) (end 252 109.5) (layer "B.SilkS") (width 4))
   (gr_line (start 59.4 48.4) (end 59.4 65.4) (layer "B.SilkS") (width 2))
-  (gr_line (start 77.276553 48.5) (end 77.276553 65.5) (layer "B.SilkS") (width 2))
+  (gr_line (start 77.276553 48.4) (end 77.276553 65.4) (layer "B.SilkS") (width 2))
   (gr_line (start 116.776553 22.259719) (end 194.9 22.259719) (layer "B.SilkS") (width 0.5))
   (gr_line (start 18 92.5) (end 57.025 92.5) (layer "B.SilkS") (width 4))
-  (gr_line (start 113 48.5) (end 113 65.5) (layer "B.SilkS") (width 2))
+  (gr_line (start 113 48.4) (end 113 65.4) (layer "B.SilkS") (width 2))
   (gr_line (start 185.449707 43.149415) (end 185.44626 41.753731) (layer "B.SilkS") (width 0.3))
   (gr_line (start 39.276553 51.509719) (end 39.276553 72.009719) (layer "B.SilkS") (width 4))
@@
   (gr_line (start 18.263277 20.75) (end 22.736724 20.75) (layer "B.SilkS") (width 4))
   (gr_arc (start 150.703042 44.158386) (mid 149.075418 43.384136) (end 148.303323 41.755489) (layer "B.SilkS") (width 0.3))
-  (gr_line (start 202.276553 48.5) (end 202.276553 65.5) (layer "B.SilkS") (width 2))
+  (gr_line (start 202.276553 48.4) (end 202.276553 65.4) (layer "B.SilkS") (width 2))
   (gr_arc (start 167.201489 41.758667) (mid 166.315072 43.486914) (end 164.49252 44.158386) (layer "B.SilkS") (width 0.3))
   (gr_line (start 27.876553 19.259719) (end 36.976553 19.259719) (layer "B.SilkS") (width 0.5))
@@
     (effects (font (size 1 1) (thickness 0.15)) (justify mirror))
   )
-  (gr_text "#Nora_kbd Switch plate DN0032 RE by @jpskenn" (at 99 73.5) (layer "B.SilkS")
+  (gr_text "#Nora_kbd Switch plate for RE, DN0032 by @jpskenn" (at 99 73.5) (layer "B.SilkS")
     (effects (font (size 1.3 1.3) (thickness 0.15)) (justify left mirror))
   )

Commit message: スイッチプレート穴サイズ、横14.2→14ｍｍに変更
Other:
- outline, holes or cut-outs redrawn
- board text added: "#Nora_kbd Switch plate for RE, DN0032(2) by @jpskenn"
- board text removed: "#Nora_kbd Switch plate for RE, DN0032 by @jpskenn"
