File: Plate_Full/keyplate/keyplate.kicad_pcb (KiCad board)
At the start: 2 copper layers, 285.4 x 94.9 mm, 3 parts

Commit message: プレート類のガーバーファイル準備
Other:
- board text added: "#Nora_kbd Switch plate for Full, DN0032 by @jpskenn"
- board text removed: "#Nora_kbd Switch plate DN0032 Full by @jpskenn"
Changed lines of the file:
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@@
   )
   (gr_line (start 139.8 25) (end 139.8 36.6) (layer "B.SilkS") (width 2))
+  (gr_line (start 59.3 48.05) (end 59.3 65.55) (layer "B.SilkS") (width 2))
   (gr_line (start 211.776553 20.759719) (end 296.776553 20.759719) (layer "B.SilkS") (width 4))
+  (gr_line (start 157.6 25) (end 157.6 36.6) (layer "B.SilkS") (width 2))
   (gr_line (start 213.5 91.75) (end 213.5 99.25) (layer "B.SilkS") (width 4))
   (gr_line (start 124.5 91.75) (end 124.5 99.25) (layer "B.SilkS") (width 4))
   (gr_arc (start 194.9 19.259719) (mid 196.4 20.759719) (end 194.9 22.259719) (layer "B.SilkS") (width 0.5))
-  (gr_line (start 166.6 47.85) (end 166.6 65.35) (layer "B.SilkS") (width 2))
+  (gr_line (start 166.6 48.05) (end 166.6 65.55) (layer "B.SilkS") (width 2))
   (gr_line (start 36.875 40.75) (end 41.625 40.75) (layer "B.SilkS") (width 2))
   (gr_arc (start 36.976553 19.259719) (mid 38.476553 20.759719) (end 36.976553 22.259719) (layer "B.SilkS") (width 0.5))
@@
   (gr_line (start 275.776553 51.009719) (end 275.776553 72.009719) (layer "B.SilkS") (width 4))
   (gr_line (start 297 92) (end 257.5 92) (layer "B.SilkS") (width 4))
+  (gr_line (start 130.8 48.05) (end 130.8 65.55) (layer "B.SilkS") (width 2))
   (gr_line (start 101.646553 91.75) (end 101.646553 99.25) (layer "B.SilkS") (width 4))
   (gr_line (start 236 91.75) (end 236 99.25) (layer "B.SilkS") (width 4))
   (gr_line (start 20.975 106.379719) (end 55.025 106.379719) (layer "B.SilkS") (width 10))
   (gr_line (start 18.026553 41.009719) (end 18.026553 68.509719) (layer "B.SilkS") (width 4))
-  (gr_line (start 146.8 91.85) (end 146.8 99.35) (layer "B.SilkS") (width 4))
+  (gr_line (start 146.8 91.75) (end 146.8 99.25) (layer "B.SilkS") (width 4))
   (gr_line (start 27.876553 22.259719) (end 36.976553 22.259719) (layer "B.SilkS") (width 0.5))
   (gr_arc (start 116.776553 22.259719) (mid 115.276553 20.759719) (end 116.776553 19.259719) (layer "B.SilkS") (width 0.5))
@@
   (gr_line (start 90.25 109.25) (end 63.25 109.25) (layer "B.SilkS") (width 4))
   (gr_line (start 191 91.75) (end 191 99.25) (layer "B.SilkS") (width 4))
-  (gr_line (start 238 48) (end 238 65.5) (layer "B.SilkS") (width 2))
+  (gr_line (start 238 48.05) (end 238 65.55) (layer "B.SilkS") (width 2))
   (gr_line (start 116.776553 19.259719) (end 194.9 19.259719) (layer "B.SilkS") (width 0.5))
   (gr_line (start 107.846553 109.379719) (end 252 109.5) (layer "B.SilkS") (width 4))
-  (gr_line (start 77.276553 48) (end 77.276553 65.5) (layer "B.SilkS") (width 2))
+  (gr_line (start 77.276553 48.05) (end 77.276553 65.55) (layer "B.SilkS") (width 2))
   (gr_line (start 121.8 25) (end 121.8 36.6) (layer "B.SilkS") (width 2))
-  (gr_line (start 95.25 48) (end 95.25 65.5) (layer "B.SilkS") (width 2))
-  (gr_line (start 113 48) (end 113 65.5) (layer "B.SilkS") (width 2))
+  (gr_line (start 95.25 48.05) (end 95.25 65.55) (layer "B.SilkS") (width 2))
+  (gr_line (start 113 48.05) (end 113 65.55) (layer "B.SilkS") (width 2))
   (gr_line (start 116.776553 22.259719) (end 194.9 22.259719) (layer "B.SilkS") (width 0.5))
-  (gr_line (start 202.25 48) (end 202.25 65.5) (layer "B.SilkS") (width 2))
+  (gr_line (start 255.7 48.05) (end 255.7 65.55) (layer "B.SilkS") (width 2))
+  (gr_line (start 202.25 48.05) (end 202.25 65.55) (layer "B.SilkS") (width 2))
   (gr_line (start 39.276553 51.509719) (end 39.276553 72.009719) (layer "B.SilkS") (width 4))
-  (gr_line (start 168.6 91.65) (end 168.6 99.15) (layer "B.SilkS") (width 4))
+  (gr_line (start 168.6 91.75) (end 168.6 99.25) (layer "B.SilkS") (width 4))
   (gr_line (start 145.000588 40.398251) (end 195.450297 40.40001) (layer "B.SilkS") (width 0.3))
   (gr_line (start 42.25 20.759719) (end 103.526553 20.759719) (layer "B.SilkS") (width 4))
   (gr_arc (start 27.876553 22.259719) (mid 26.376553 20.759719) (end 27.876553 19.259719) (layer "B.SilkS") (width 0.5))
   (gr_line (start 297.026553 41.009719) (end 297.026553 69) (layer "B.SilkS") (width 4))
-  (gr_line (start 220.25 48) (end 220.25 65.5) (layer "B.SilkS") (width 2))
+  (gr_line (start 220.25 48.05) (end 220.25 65.55) (layer "B.SilkS") (width 2))
   (gr_line (start 57.5 92) (end 18 92) (layer "B.SilkS") (width 4))
-  (gr_line (start 148.6 48) (end 148.6 65.5) (layer "B.SilkS") (width 2))
+  (gr_line (start 148.6 48.05) (end 148.6 65.55) (layer "B.SilkS") (width 2))
   (gr_arc (start 195.499124 38.6) (mid 196.4 39.525104) (end 195.450297 40.40001) (layer "B.SilkS") (width 0.3))
   (gr_line (start 18.263277 20.75) (end 22.736724 20.75) (layer "B.SilkS") (width 4))
   (gr_line (start 79.5 91.75) (end 79.5 99.25) (layer "B.SilkS") (width 4))
+  (gr_line (start 184.4 48.05) (end 184.4 65.55) (layer "B.SilkS") (width 2))
   (gr_line (start 27.876553 19.259719) (end 36.976553 19.259719) (layer "B.SilkS") (width 0.5))
   (gr_line (start 175.4 25) (end 175.4 36.6) (layer "B.SilkS") (width 2))
@@
     (effects (font (size 1 1) (thickness 0.15)) (justify mirror))
   )
-  (gr_text "#Nora_kbd Switch plate DN0032 Full by @jpskenn" (at 95 73.6) (layer "B.SilkS")
+  (gr_text "#Nora_kbd Switch plate for Full, DN0032 by @jpskenn" (at 97.6 73.6) (layer "B.SilkS")
     (effects (font (size 1.3 1.3) (thickness 0.15)) (justify left mirror))
   )

Commit message: スイッチプレート穴サイズ、横14.2→14ｍｍに変更
Other:
- outline, holes or cut-outs redrawn
- board text added: "#Nora_kbd Switch plate for Full, DN0032(2) by @jpskenn"
- board text removed: "#Nora_kbd Switch plate for Full, DN0032 by @jpskenn"
